Commit message: first test on real robot

File: blue_arm_description/urdf/blue_arm.xacro (robot description, xacro)
@@ -111,5 +111,5 @@
       upper="3.1415926"
       effort="1000"
-      velocity="6" />
+      velocity="0.26" />
   </joint>
   <link
@@ -166,8 +166,8 @@
       xyz="0 -1 0" />
     <limit
-      lower="-3"
+      lower="0"
       upper="3.1415926"
       effort="1000"
-      velocity="6" />
+      velocity="0.26" />
   </joint>
   <link
@@ -222,10 +222,10 @@
       link="link_3" />
     <axis
-      xyz="-1 0 0" />
+      xyz="1 0 0" />
     <limit
       lower="-3.1415926"
       upper="3.1415926"
       effort="1000"
-      velocity="6" />
+      velocity="0.26" />
   </joint>
   <link
@@ -280,10 +280,10 @@
       link="link_4" />
     <axis
-      xyz="0 1 0" />
-    <limit
-      lower="0"
-      upper="3.1415926"
-      effort="1000"
-      velocity="6" />
+      xyz="0 -1 0" />
+    <limit
+      lower="-3.1415926"
+      upper="0"
+      effort="1000"
+      velocity="0.26" />
   </joint>
   <link
@@ -338,10 +338,10 @@
       link="link_5" />
     <axis
-      xyz="-1 0 0" />
+      xyz="1 0 0" />
     <limit
       lower="-3.1415926"
       upper="3.1415926"
       effort="1000"
-      velocity="6" />
+      velocity="0.26" />
   </joint>
   <link
@@ -396,10 +396,10 @@
       link="link_6" />
     <axis
-      xyz="0 1 0" />
+      xyz="0 -1 0" />
     <limit
       lower="-1.7"
       upper="1.7"
       effort="1000"
-      velocity="6" />
+      velocity="0.26" />
   </joint>
   <link
@@ -437,10 +437,10 @@
       link="link_7" />
     <axis
-      xyz="-1 0 0" />
+      xyz="1 0 0" />
     <limit
       lower="-3.1415926"
       upper="3.1415926"
       effort="1000"
-      velocity="6" />
+      velocity="0.26" />
   </joint>
 </robot>
